File: teensy4_ramps.kicad_pcb (KiCad board)
At the start: 4 copper layers, 101.6 x 53.3 mm, 18 parts, among them J1 USB_B_Mini, J2 Barrel_Jack_Switch, J3 Conn_01x03, U1 Teensy4.1, U2 AOZ1282CI

Commit message: update
Parts:
- C5: value 33uF, 16V -> 22uF, 16V; footprint Capacitor_SMD:CP_Elec_5x5.4 -> Capacitor_SMD:CP_Elec_4x5.3
- D2: value B260A-13-F -> BAT60AE6327; footprint Diode_SMD:D_SMA -> Diode_SMD:D_SOD-323
- L1: value 22uH -> 4.7uH
- U2: value AOZ1282CI -> AOZ1280
Routing:
- net Net-(C3-Pad1): track 3.34 -> 0.00 mm
- net GND: track 22.7 -> 25.7 mm, vias 24 -> 27
- net /Z_STEP: track 93.9 -> 94.9 mm
- net /Z_DIR: track 90.2 -> 91.3 mm
- net /E0_DIR: track 110.2 -> 110.7 mm
Other:
- board size 101.6 x 53.3 mm -> 99.1 x 53.3 mm
