File: teensy4_ramps.sch (KiCad schematic (older format))
At the start: 18 parts, among them J1 USB_B_Mini, J2 Barrel_Jack_Switch, J3 Conn_01x03, U1 Teensy4.1, U2 AOZ1282CI

Commit message: update
Parts:
- C5: value 33uF, 16V -> 22uF, 16V; footprint Capacitor_SMD:CP_Elec_5x5.4 -> Capacitor_SMD:CP_Elec_4x5.3
- D2: value B260A-13-F -> BAT60AE6327; footprint Diode_SMD:D_SMA -> Diode_SMD:D_SOD-323
- L1: value 22uH -> 4.7uH
- U2: value AOZ1282CI -> AOZ1280
Changed lines of the file:
@@
 P 4050 7200
 F 0 "D2" V 4050 7000 50  0000 L CNN
-F 1 "B260A-13-F" H 3850 7300 50  0000 L CNN
-F 2 "Diode_SMD:D_SMA" H 4050 7200 50  0001 C CNN
+F 1 "BAT60AE6327" H 3850 7300 50  0000 L CNN
+F 2 "Diode_SMD:D_SOD-323" H 4050 7200 50  0001 C CNN
 F 3 "~" H 4050 7200 50  0001 C CNN
 	1    4050 7200
@@
 P 3400 6800
 F 0 "U2" H 3400 7167 50  0000 C CNN
-F 1 "AOZ1282CI" H 3400 7076 50  0000 C CNN
+F 1 "AOZ1280" H 3400 7076 50  0000 C CNN
 F 2 "Package_TO_SOT_SMD:SOT-23-6" H 4100 6550 50  0001 C CNN
 F 3 "http://aosmd.com/res/data_sheets/AOZ1282CI.pdf" H 3150 6550 50  0001 C CNN
@@
 P 5250 7100
 F 0 "C5" H 5365 7146 50  0000 L CNN
-F 1 "33uF, 16V" H 5365 7055 50  0000 L CNN
-F 2 "Capacitor_SMD:CP_Elec_5x5.4" H 5250 7100 50  0001 C CNN
+F 1 "22uF, 16V" H 5365 7055 50  0000 L CNN
+F 2 "Capacitor_SMD:CP_Elec_4x5.3" H 5250 7100 50  0001 C CNN
 F 3 "~" H 5250 7100 50  0001 C CNN
 	1    5250 7100
@@
 P 4400 6800
 F 0 "L1" V 4590 6800 50  0000 C CNN
-F 1 "22uH" V 4499 6800 50  0000 C CNN
+F 1 "4.7uH" V 4499 6800 50  0000 C CNN
 F 2 "Inductor_SMD:L_Taiyo-Yuden_NR-50xx" H 4400 6800 50  0001 C CNN
 F 3 "~" H 4400 6800 50  0001 C CNN
